Commit message: docker support added

File: project_apr_pkg/model/omni_58mm.xacro (robot description, xacro)
@@ -42,5 +42,5 @@
     </link>
     <gazebo reference="${name}">
-        <material>Gazebo/White</material>
+        <material>Gazebo/Grey</material>
         <!-- friction coeff along the friction axis -->
         <mu1>0.0</mu1>
